File: project/project.kicad_sch (KiCad schematic)
At the start: 148 parts, among them J1 2.54mm 1*20P, J2 2.54mm 1*20P, SW1 KMR221GLFS, SW2 KMR221GLFS, U1 XC7A100T-FGG484, U2 TPS65261RHBR, U3 FT2232HL, U4 93LC46B-E/SN, U5 TPD2EUSB30, U6 W25Q256JVFIQT, U7 IS66WVH16M8DALL-166B1LI

Commit message: new
Parts:
- added Q1: AO3400A, lcsc_footprints:C20917_SOT-23-3_L2_9-W1_3-P1_90-LS2_4-BR, symbol lcsc_imported:AO3400A
- C1, C11, C12, C14, C16, C17, C19, C21, C22, C23, C27, C29, C31, C32, C33, C34, C35, C36, C37, C38, C39, C4, C42, C48, C49, C5, C50, C51, C52, C53, C54, C55, C60, C61, C62, C63, C64, C67, C69, C73, C74, C75, C76, C77, C78, C79, C80, C81, C82, C84, C9: footprint (none) -> Capacitor_SMD:C_0402_1005Metric
- C10: value 1µF -> 10µF; footprint (none) -> Capacitor_SMD:C_0805_2012Metric
- C13, C15, C18, C2, C20, C3, C6, C7, C8: footprint (none) -> Capacitor_SMD:C_0805_2012Metric
- C24: footprint lcsc_footprints:C5280582_OSC-SMD_4P-L3_2-W2_5-BL -> Capacitor_SMD:C_0805_2012Metric
- C25: footprint lcsc_footprints:C5280582_OSC-SMD_4P-L3_2-W2_5-BL -> Capacitor_SMD:C_0402_1005Metric
- C26, C28, C30, C41, C43, C44, C45, C46, C47, C58, C59, C65, C70, C72, C83, C85: footprint (none) -> Capacitor_SMD:C_0603_1608Metric
- C40: footprint (none) -> lcsc_footprints:C314600_C1210
- C56, C66, C68, C71, C86: footprint (none) -> Capacitor_SMD:C_1206_3216Metric
- C57: footprint (none) -> lcsc_footprints:C15008_C1206
- FB1, FB2: footprint (none) -> lcsc_footprints:C1002_L0603
- L1: footprint (none) -> lcsc_footprints:C160951_IND-SMD_L6_0-W6_0
- L2, L3: footprint (none) -> lcsc_footprints:C162577_IND-SMD_L5_0-W5_0
- R1, R10, R11, R12, R13, R14, R15, R16, R17, R18, R2, R22, R23, R24, R25, R26, R27, R3, R33, R37, R38, R39, R4, R40, R5, R6, R7, R8, R9: footprint (none) -> Resistor_SMD:R_0402_1005Metric
- R19, R20, R21, R36, R41, R42: footprint Resistor_THT:R_Array_SIP4 -> Resistor_SMD:R_0402_1005Metric
- R28, R29, R30, R31, R32, R34: value 10kΩ -> 4.7kΩ; footprint Resistor_THT:R_Array_SIP4 -> Resistor_SMD:R_0402_1005Metric
- R35: value 680Ω -> 130Ω; footprint Resistor_THT:R_Array_SIP4 -> Resistor_SMD:R_0402_1005Metric
- U2: footprint RHB0032E -> ul_TPS65261RHBR:RHB0032E
- U4: footprint SOIC8-N_MC_MCH -> ul_93LC46B-E-SN:SOIC8-N_MC_MCH
- U7: footprint BGA24_IS66_ISI -> ul_IS66WVH16M8DALL-166B1LI:BGA24_IS66_ISI
Connections:
- net GNDA is gone; now on net GND: C12.2, C17.2, C21.2, C22.2, C23.2, C4.2, R11.2, R14.2, R3.2, R4.1, R6.1, U2.21 (AGND), U3.10 (AGND)
- net FTDI_JTAG_TCK: now also U1.V12 (TCK_0); no longer U1.R13 (TDI_0)
- net FTDI_JTAG_TDI: now also U1.R13 (TDI_0); no longer U1.U13 (TDO_0)
- net FTDI_JTAG_TDO: now also U1.U13 (TDO_0); no longer U1.T13 (TMS_0)
- net FTDI_JTAG_TMS: now also U1.T13 (TMS_0); no longer U1.V12 (TCK_0)
- net GND: now also J1.10, J1.15, J1.20, J1.5, J2.10, J2.15, J2.20, J2.5, U2.33 (PAD), Q1.2 (S); no longer LED1.1 (K)
- net USB_DN: now also USB1.A7 (DN1); no longer USB1.A6 (DP1)
- net USB_DP: now also USB1.A6 (DP1); no longer USB1.A7 (DN1)
- net VBUS: now also C6.2, C7.2, C8.2, C9.2, R5.1, U2.12 (PVIN2), U2.13 (PVIN3), U2.28 (PVIN1), U2.29 (VIN)
- net VCC3V3: now also R35.1, U1.U22 (IO_L3P_T0_DQS_PUDC_B_14)
- net FPGA_RESET: now reaches R42.2, U7.A4 (RESET#)
- net FPGA_RESET: now also U1.K1 (IO_L7P_T1_AD6P_35)
- net at U1.J6 (IO_L17N_T2_35): no longer J2.10
- net at U1.R1 (IO_L20P_T3_35): no longer J2.15
- net at U1.N2 (IO_L22N_T3_35): no longer J2.20
- net at U1.M1 (IO_L15P_T2_DQS_35): no longer J2.5
- net at U1.AA19 (IO_L15P_T2_DQS_RDWR_B_14): no longer J1.15
- net at U1.AB18 (IO_L17N_T2_A13_D29_14): no longer J1.20
- net at U1.AB21 (IO_L10P_T1_D14_14): no longer J1.5
- net at J1.9: now also U1.W20 (IO_L12N_T1_MRCC_14); no longer U1.W19 (IO_L12P_T1_MRCC_14)
- net FPGA_CS: now reaches R41.2, U7.A3 (CS#)
- net FPGA_CS: now also U1.F1 (IO_L5N_T0_AD13N_35)
- net at U7.C5 (RFU): no longer U1.D2 (IO_L4N_T0_35)
- net at U1.G11 (DONE_0): now also Q1.1 (G); no longer R35.1
- net FPGA_PSC_P: no longer names the net of U7.B5 (RFU)
- net FPGA_PSC_P: no longer U1.E2 (IO_L4P_T0_35)
- net OSC_12MHZ renamed OSC_12
- net OSC_12: now also U1.W19 (IO_L12P_T1_MRCC_14)
- new net: LED1.1 (K), Q1.3 (D)
- no-connect marks 101 -> 116
Other:
- note added: "1.8V I/O"
- moved on the sheet: C1, C10, C11, C12, C13, C14, C15, C16, C17, C18, C19, C2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
